File: rs_lever/rs_lever.kicad_pcb (KiCad board)
At the start: 2 copper layers, 47 x 44 mm, 8 parts, among them J1 SOC, J2 PIN, SW1 SW_SPDT

Commit message: update
Parts:
- removed the G*** at (66.0, 66.0)

Commit message: update
Parts:
- added TP3: BATTERY1_{-}, TestPoint:TestPoint_THTPad_D2.5mm_Drill1.2mm, F.Cu at (65.0, 40.0)
- added TP4: BATTERY2_{+}, TestPoint:TestPoint_THTPad_D2.5mm_Drill1.2mm, F.Cu at (44.0, 60.0)
- TP1: value BATTERY_{+} -> BATTERY1_{+}
- TP2: value BATTERY_{-} -> BATTERY2_{-}
- moved TP2 23.1 mm to (64.0, 60.0)
- moved TP1 0.50 mm to (45.0, 40.0)
Routing:
- net Net-(TP3-Pad1): track 0.00 -> 29.3 mm
- net /OUT: track 29.7 -> 30.7 mm
- net Net-(D1-A): track 10.3 -> 9.79 mm

Commit message: fixed_lever
Parts:
- added D2: 1N4007, Diode_THT:D_DO-35_SOD27_P7.62mm_Horizontal, F.Cu at (32.5, 38.3)
- moved TP1 1.41 mm to (46.0, 39.0)
- moved TP3 1.41 mm to (66.0, 39.0)
- moved TP2 1.00 mm to (64.0, 59.0)
- moved TP4 1.00 mm to (44.0, 59.0)
Connections:
- SW1 pad 2: /OUT -> Net-(D2-A)
Routing:
- net Net-(D2-A): track 0.00 -> 30.6 mm
- net /OUT: track 30.7 -> 21.8 mm
- net Net-(D1-A): track 9.79 -> 11.2 mm
- net Net-(TP3-Pad1): track 29.3 -> 30.3 mm
