File: rs_lamp/rs_lamp.kicad_pcb (KiCad board)
At the start: 2 copper layers, 47 x 44 mm, 7 parts, among them J1 SOC, J2 PIN, Q1 2N7000

Commit message: fixed_sensor_2
Parts:
- moved Q1 17.4 mm to (44.0, 54.2)
- moved R2 13.0 mm to (60.0, 53.3), turned to 90 degrees
- moved G*** 9.19 mm to (66.0, 56.0)
- moved R4 6.79 mm to (32.7, 46.0), turned to 0 degrees
Routing:
- net GND: track 42.1 -> 0.00 mm
- net /IN: track 36.2 -> 25.7 mm
- net Net-(Q1-D): track 12.5 -> 17.4 mm
- net Net-(D1-K): track 12.0 -> 11.1 mm
Other:
- board size 47 x 44 mm -> 47 x 24 mm
