File: rs_light_sensor/rs_light_sensor.kicad_pcb (KiCad board)
At the start: 2 copper layers, 47 x 44 mm, 7 parts, among them J1 SOC, J2 PIN, Q1 2N7000

Commit message: update
Parts:
- added D2: 1N4007, Diode_THT:D_DO-35_SOD27_P7.62mm_Horizontal, F.Cu at (40.2, 60.0)
- added R3: 10k, Resistor_THT:R_Axial_DIN0207_L6.3mm_D2.5mm_P7.62mm_Horizontal, F.Cu at (39.7, 55.0)
- added TP1: BATTERY_{+}, TestPoint:TestPoint_THTPad_D2.5mm_Drill1.2mm, F.Cu at (46.0, 37.0)
- added TP2: BATTERY_{-}, TestPoint:TestPoint_THTPad_D2.5mm_Drill1.2mm, F.Cu at (52.5, 37.0)
- D1: value LED -> 1N4007; footprint LED_THT:LED_D3.0mm -> Diode_THT:D_DO-35_SOD27_P7.62mm_Horizontal
- R2: value 330 -> CDS; footprint Resistor_THT:R_Axial_DIN0207_L6.3mm_D2.5mm_P7.62mm_Horizontal -> OptoDevice:R_LDR_D6.4mm_P3.4mm_Vertical
- R4: value 100k -> 510k
- moved Q1 23.0 mm to (54.8, 60.1), turned to 180 degrees
- moved R2 16.7 mm to (48.3, 50.0), turned to 0 degrees
- moved D1 14.5 mm to (35.5, 48.3), turned to 90 degrees
- moved G*** 13.7 mm to (65.0, 50.0)
- moved R4 1.29 mm to (40.2, 44.0), turned to 0 degrees
Connections:
- D1 pad 1: Net-(D1-K) -> +5V
- D1 pad 2: +5V -> Net-(D1-A)
- J1 pad 2: /IN -> /OUT
- J2 pad 2: /IN -> /OUT
- Q1 pad 2: /IN -> Net-(Q1-G)
- Q1 pad 3: Net-(Q1-D) -> Net-(D2-A)
- R2 pad 1: Net-(Q1-D) -> Net-(Q1-G)
- R2 pad 2: Net-(D1-K) -> GND
- R4 pad 1: /IN -> +5V
- R4 pad 2: GND -> Net-(Q1-G)
Routing:
- net GND: track 42.1 -> 0.00 mm
- net /IN: track 36.2 -> 0.00 mm
- net /OUT: track 0.00 -> 20.8 mm
- net Net-(Q1-G): track 0.00 -> 18.5 mm
- net Net-(Q1-D): track 12.5 -> 0.00 mm
- net Net-(D1-K): track 12.0 -> 0.00 mm
- net Net-(D1-A): track 0.00 -> 12.0 mm
- net Net-(D2-A): track 0.00 -> 9.69 mm
- net +5V: track 22.6 -> 21.7 mm
Other:
- board text removed: "A"
- board text removed: "K"

Commit message: fixed_sensor
Parts:
- removed D1: 1N4007, Diode_THT:D_DO-35_SOD27_P7.62mm_Horizontal
- removed TP1: BATTERY_{+}, TestPoint:TestPoint_THTPad_D2.5mm_Drill1.2mm
- removed TP2: BATTERY_{-}, TestPoint:TestPoint_THTPad_D2.5mm_Drill1.2mm
- added J3: IN_{PIN}, Connector_PinHeader_2.54mm:PinHeader_1x03_P2.54mm_Horizontal, B.Cu at (70.5, 57.0)
- added J4: IN_{SOC}, Connector_PinSocket_2.54mm:PinSocket_1x03_P2.54mm_Horizontal, B.Cu at (64.5, 43.0)
- J1: value SOC -> OUT_{SOC}
- J2: value PIN -> OUT_{PIN}
- moved G*** 22.3 mm to (48.5, 35.0)
Routing:
- net +5V: track 21.7 -> 58.9 mm
- net /IN: track 0.00 -> 13.4 mm
- net Net-(D1-A): track 12.0 -> 0.00 mm
- net /OUT: track 20.8 -> 21.5 mm
Other:
- board size 47 x 44 mm -> 50 x 44 mm

Commit message: fixed_sensor_2
Parts:
- removed J1: OUT_{SOC}, Connector_PinSocket_2.54mm:PinSocket_1x03_P2.54mm_Horizontal
- J2: footprint Connector_PinHeader_2.54mm:PinHeader_1x03_P2.54mm_Horizontal -> Connector_PinHeader_2.54mm:PinHeader_1x03_P2.54mm_Vertical
- moved D2 17.5 mm to (33.2, 44.0)
- moved G*** 17.3 mm to (61.0, 47.0)
- moved R4 5.78 mm to (45.9, 43.0)
- moved Q1 5.58 mm to (59.0, 56.5)
- moved R3 4.91 mm to (34.9, 56.0)
- moved J2 2.50 mm to (27.0, 43.0)
Routing:
- net Net-(D2-A): track 9.69 -> 26.9 mm
- net /OUT: track 21.5 -> 6.81 mm
- net GND: track 0.00 -> 5.31 mm
- net Net-(Q1-G): track 18.5 -> 21.7 mm
- net +5V: track 58.9 -> 57.1 mm
Other:
- board size 50 x 44 mm -> 50 x 24 mm
