File: rs_torch/rs_torch.kicad_pcb (KiCad board)
At the start: 2 copper layers, 50 x 50 mm, 20 parts, among them J1 INPUT_SOC, J2 INPUT_PIN, J3 OUTPUT_PIN, J4 OUTPUT_SOC, J5 INPUT2_PIN, J6 INPUT2_SOC, J7 INPUT3_SOC, J8 INPUT3_PIN, Q1 2N7000, Q2 2N7000

Commit message: correction
Parts:
- TP1: value LED_{A} -> LED_A
- TP2: value LED_{K} -> LED_K
- moved J5 9.00 mm to (57.0, 29.5)
- moved J6 9.00 mm to (43.0, 35.5)
- moved J7 9.00 mm to (57.0, 64.5)
- moved J8 9.00 mm to (43.0, 70.5)
- moved R5 6.02 mm to (61.0, 62.5)
- moved TP1 4.27 mm to (56.0, 52.5)
- moved TP2 4.03 mm to (56.0, 49.0)
- moved D1 3.16 mm to (66.1, 57.0)
- moved J3 0.50 mm to (70.5, 57.0)
Connections:
- J5 pad 1: +5V -> GND
- J5 pad 3: GND -> +5V
- J6 pad 1: +5V -> GND
- J6 pad 3: GND -> +5V
- J7 pad 1: +5V -> GND
- J7 pad 3: GND -> +5V
- J8 pad 1: +5V -> GND
- J8 pad 3: GND -> +5V
Routing:
- net GND: track 143.7 -> 0.00 mm, vias 4 -> 0
- net /LED_A: track 29.4 -> 9.49 mm
- net Net-(D1-A): track 32.3 -> 42.1 mm
- net /LED_K: track 7.14 -> 4.08 mm
- net /OUT: track 21.1 -> 18.8 mm
- net /IN: track 82.5 -> 80.4 mm
- net +5V: track 93.0 -> 94.2 mm
Other:
- board text added: "OUT"

Commit message: fixed_torch
Parts:
- removed the G*** at (36.0, 36.0)
- removed the G*** at (34.0, 66.0)
- added D2: 11EQS06, Diode_THT:D_DO-41_SOD81_P10.16mm_Horizontal, F.Cu at (33.0, 31.0)
- added D3: 11EQS06, Diode_THT:D_DO-41_SOD81_P10.16mm_Horizontal, F.Cu at (38.5, 30.9)
- added D4: 11EQS06, Diode_THT:D_DO-41_SOD81_P10.16mm_Horizontal, F.Cu at (31.9, 65.5)
- added G***: LOGO, _footprints:eleken_logo, F.Cu at (64.5, 35.5)
- D1: value 1N4007 -> 11EQS06
Connections:
- J1 pad 2: /IN -> Net-(D2-A)
- J2 pad 2: /IN -> Net-(D2-A)
- J5 pad 2: /IN -> Net-(D3-A)
- J6 pad 2: /IN -> Net-(D3-A)
- J7 pad 2: /IN -> Net-(D4-A)
- J8 pad 2: /IN -> Net-(D4-A)
Routing:
- net /IN: track 80.4 -> 42.6 mm
- net Net-(D3-A): track 0.00 -> 22.7 mm
- net Net-(D4-A): track 0.00 -> 19.8 mm
- net Net-(D2-A): track 0.00 -> 19.2 mm
