File: rs_torch/rs_torch.kicad_sch (KiCad schematic)
At the start: 18 parts, among them J1 INPUT_SOC, J2 INPUT_PIN, J3 OUTPUT_PIN, J4 OUTPUT_SOC, J5 INPUT2_PIN, J6 INPUT2_SOC, J7 INPUT3_SOC, J8 INPUT3_PIN, Q1 2N7000, Q2 2N7000

Commit message: correction
Connections:
- net +5V: now also J5.3 (Pin_3), J6.3 (Pin_3), J7.3 (Pin_3), J8.3 (Pin_3); no longer J5.1 (Pin_1), J6.1 (Pin_1), J7.1 (Pin_1), J8.1 (Pin_1)
- net GND: now also J5.1 (Pin_1), J6.1 (Pin_1), J7.1 (Pin_1), J8.1 (Pin_1); no longer J5.3 (Pin_3), J6.3 (Pin_3), J7.3 (Pin_3), J8.3 (Pin_3)
Other:
- moved on the sheet: J6, J8
Changed lines of the file:
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@@
 		)
 		(instances
-			(project "eleken"
+			(project "rs_torch"
 				(path "/d626508b-3053-4ce9-abdf-fc345aae31e1"
 					(reference "D1")
@@
 		)
 		(instances
-			(project "eleken"
+			(project "rs_torch"
 				(path "/d626508b-3053-4ce9-abdf-fc345aae31e1"
 					(reference "R5")
@@
 		)
 		(instances
-			(project "eleken"
+			(project "rs_torch"
 				(path "/d626508b-3053-4ce9-abdf-fc345aae31e1"
 					(reference "J4")
@@
 		)
 		(instances
-			(project "eleken"
+			(project "rs_torch"
 				(path "/d626508b-3053-4ce9-abdf-fc345aae31e1"
 					(reference "R3")
@@
 		)
 		(instances
-			(project "eleken"
+			(project "rs_torch"
 				(path "/d626508b-3053-4ce9-abdf-fc345aae31e1"
 					(reference "R4")
@@
 		)
 		(instances
-			(project "eleken"
+			(project "rs_torch"
 				(path "/d626508b-3053-4ce9-abdf-fc345aae31e1"
 					(reference "#PWR04")
@@
 		)
 		(instances
-			(project "eleken"
+			(project "rs_torch"
 				(path "/d626508b-3053-4ce9-abdf-fc345aae31e1"
 					(reference "R2")
@@
 		)
 		(instances
-			(project "eleken"
+			(project "rs_torch"
 				(path "/d626508b-3053-4ce9-abdf-fc345aae31e1"
 					(reference "J2")
@@
 		)
 		(instances
-			(project "eleken"
+			(project "rs_torch"
 				(path "/d626508b-3053-4ce9-abdf-fc345aae31e1"
 					(reference "R1")
@@
 		(lib_id "Connector:Conn_01x03_Socket")
 		(at 90.17 27.94 0)
-		(mirror x)
 		(unit 1)
 		(body_style 1)
@@
 		(dnp no)
 		(property "Reference" "J7"
-			(at 92.964 30.226 0)
+			(at 92.964 25.654 0)
 			(show_name no)
 			(do_not_autoplace no)
@@
 		)
 		(property "Value" "INPUT3_SOC"
-			(at 91.694 26.924 0)
+			(at 91.694 28.956 0)
 			(show_name no)
 			(do_not_autoplace no)
@@
 		)
 		(instances
-			(project "eleken"
+			(project "rs_torch"
 				(path "/d626508b-3053-4ce9-abdf-fc345aae31e1"
 					(reference "J7")
@@
 		)
 		(instances
-			(project "eleken"
+			(project "rs_torch"
 				(path "/d626508b-3053-4ce9-abdf-fc345aae31e1"
 					(reference "#PWR03")
@@
 		)
 		(instances
-			(project "eleken"
+			(project "rs_torch"
 				(path "/d626508b-3053-4ce9-abdf-fc345aae31e1"
 					(reference "J1")
@@
 		)
 		(instances
-			(project "eleken"
+			(project "rs_torch"
 				(path "/d626508b-3053-4ce9-abdf-fc345aae31e1"
 					(reference "#PWR01")
@@
 		)
 		(instances
-			(project "eleken"
+			(project "rs_torch"
 				(path "/d626508b-3053-4ce9-abdf-fc345aae31e1"
 					(reference "Q1")
@@
 		)
 		(instances
-			(project "eleken"
+			(project "rs_torch"
 				(path "/d626508b-3053-4ce9-abdf-fc345aae31e1"
 					(reference "#PWR05")
@@
 		(lib_id "Connector:Conn_01x03_Pin")
 		(at 52.07 27.94 0)
-		(mirror x)
 		(unit 1)
 		(body_style 1)
@@
 		(dnp no)
 		(property "Reference" "J5"
-			(at 48.26 30.734 0)
+			(at 48.26 25.146 0)
 			(show_name no)
 			(do_not_autoplace no)
@@
 		)
 		(property "Value" "INPUT2_PIN"
-			(at 45.72 27.686 0)
+			(at 45.72 28.194 0)
 			(show_name no)
 			(do_not_autoplace no)
@@
 		)
 		(instances
-			(project "eleken"
+			(project "rs_torch"
 				(path "/d626508b-3053-4ce9-abdf-fc345aae31e1"
 					(reference "J5")
@@
 		)
 		(instances
-			(project "eleken"
+			(project "rs_torch"
 				(path "/d626508b-3053-4ce9-abdf-fc345aae31e1"
 					(reference "#PWR02")
@@
 	(symbol
 		(lib_id "Connector:Conn_01x03_Socket")
-		(at 52.07 35.56 0)
-		(mirror y)
+		(at 52.07 35.56 180)
 		(unit 1)
 		(body_style 1)
@@
 		(dnp no)
 		(property "Reference" "J6"
-			(at 49.276 33.274 0)
+			(at 49.276 37.846 0)
 			(show_name no)
 			(do_not_autoplace no)
@@
 		)
 		(property "Value" "INPUT2_SOC"
-			(at 50.8 36.8299 0)
+			(at 50.8 34.2901 0)
 			(show_name no)
 			(do_not_autoplace no)
@@
 		)
 		(instances
-			(project "eleken"
+			(project "rs_torch"
 				(path "/d626508b-3053-4ce9-abdf-fc345aae31e1"
 					(reference "J6")
@@
 		)
 		(instances
-			(project "eleken"
+			(project "rs_torch"
 				(path "/d626508b-3053-4ce9-abdf-fc345aae31e1"
 					(reference "#PWR06")
@@
 		)
 		(instances
-			(project "eleken"
+			(project "rs_torch"
 				(path "/d626508b-3053-4ce9-abdf-fc345aae31e1"
 					(reference "J3")
@@
 		)
 		(instances
-			(project "eleken"
+			(project "rs_torch"
 				(path "/d626508b-3053-4ce9-abdf-fc345aae31e1"
 					(reference "Q2")
@@
 	(symbol
 		(lib_id "Connector:Conn_01x03_Pin")
-		(at 90.17 35.56 0)
-		(mirror y)
+		(at 90.17 35.56 180)
 		(unit 1)
 		(body_style 1)
@@
 		(dnp no)
 		(property "Reference" "J8"
-			(at 93.98 32.766 0)
+			(at 93.98 38.354 0)
 			(show_name no)
 			(do_not_autoplace no)
@@
 		)
 		(property "Value" "INPUT3_PIN"
-			(at 97.282 36.322 0)
+			(at 97.282 34.798 0)
 			(show_name no)
 			(do_not_autoplace no)
@@
 		)
 		(instances
-			(project "eleken"
+			(project "rs_torch"
 				(path "/d626508b-3053-4ce9-abdf-fc345aae31e1"
 					(reference "J8")
@@
 		)
 		(instances
-			(project "eleken"
+			(project "rs_torch"
 				(path "/d626508b-3053-4ce9-abdf-fc345aae31e1"
 					(reference "TP2")
@@
 		)
 		(instances
-			(project "eleken"
+			(project "rs_torch"
 				(path "/d626508b-3053-4ce9-abdf-fc345aae31e1"
 					(reference "TP1")

Commit message: fixed_torch
Parts:
- added D2, D3, D4: 11EQS06, Diode_THT:D_DO-41_SOD81_P10.16mm_Horizontal, symbol Diode:1N4007
- D1: value 1N4007 -> 11EQS06
Connections:
- net IN: now also D2.1 (K), D3.1 (K), D4.1 (K); no longer J1.2 (Pin_2), J2.2 (Pin_2), J5.2 (Pin_2), J6.2 (Pin_2), J7.2 (Pin_2), J8.2 (Pin_2)
- new net: D4.2 (A), J7.2 (Pin_2), J8.2 (Pin_2)
- new net: D2.2 (A), J1.2 (Pin_2), J2.2 (Pin_2)
- new net: D3.2 (A), J5.2 (Pin_2), J6.2 (Pin_2)
Other:
- moved on the sheet: J3, J4, J7, J8, TP1, TP2
